File: supply_interface/supply_interface.kicad_sch (KiCad schematic)
At the start: 59 parts, among them J1 39-28-1243, J10 MBES-152, J11 MBES-152, J12 MBES-152, J13 MBES-152, J15 3-641215-2, J2 39-28-1043, J3 MBES-152, J4 MBES-152, J5 282837-3, J6 MBES-152, J7 39-28-1043, J8 MBES-152, J9 MBES-152

Commit message: Update supply interface KiCad project and external libraries
Parts:
- removed F11, F7: 3413.0329.22, FUSC3216X60N, symbol 3413.0329.22:3413.0329.22
- removed F4: SF-1206S1000R-2, FUSC3216X90N, symbol SF-1206S1000R-2:SF-1206S1000R-2
- removed F5: 049401.5NRHF, 0494015NRHF, symbol 049401_5NRHF:049401.5NRHF
- removed F6: 0494002.NRHF, FUSC1608X30N, symbol 0494002_NRHF:0494002.NRHF
- removed J11, J3: MBES-152, CONN_MBES-152_ALT, symbol MBES-152:MBES-152
- removed J2, J7: 39-28-1043, 39-28-1043, symbol 39-28-1043:39-28-1043
- removed PS1: TEL_15-1215N, TEL151215N, symbol TEL_15-1215N:TEL_15-1215N
- added C5, C7: 22 uF, CAPC2012X145N, symbol CL21A226MAYNNNE:CL21A226MAYNNNE
- added C6: 220 uF, CAPAE1050X1050N, symbol MAL215097001E3:MAL215097001E3
- added C8: 100 uF, CAPPM7343X310N, symbol T55D107M025C0060:T55D107M025C0060
- added D8: DFLT27A-7, DFLT27A7, symbol DFLT27A-7:DFLT27A-7
- added F12: 20A F.B, FUS_CB_3216FF, symbol TR/3216FF20-R:TR_3216FF20-R
- added F13: 6A S.B, FUSC1608X95N, symbol SF-0603SA600M-2:SF-0603SA600M-2
- added F14: 1.6 S.B, FUSC1608X55N, symbol SF-0603S160-2:SF-0603S160-2
- added F4, F5, F6: 4A S.B, FUSC1005X61N, symbol SF-0402S400M-2:SF-0402S400M-2
- added F7: 8A S.B, 0ABB8000TM, symbol 0ABB-8000-TM:0ABB-8000-TM
- added J14: 39-28-1043, 39-28-1043, symbol 39-28-1043:39-28-1043
- added J2: 39-28-1063, 39-28-1063, symbol 39-28-1063:39-28-1063
- added J7: 39-28-1083, 39-28-1083, symbol 39-28-1083:39-28-1083
- added PS3: THN_30-1215, THN302415, symbol THN 30-1215:THN_30-1215
- added PS4: IRE-24_5-Q12N-C, IRE245Q12NC, symbol IRE-24/5-Q12N-C:IRE-24_5-Q12N-C
- C3: value CL21A226MAYNNNE -> 22 uF
- F1: value SF-0603S100-2 -> 0.8 A S.B
- F10, F8: value 0ABA-0200-TN -> 0.2A S.B
- F2: value 3403.0157.24 -> 0.125 A S.B
- F3: value SF-1206S300-2 -> 3A S.B
- F9: value SF-0603SP080-2 -> 0.8 A S.B
Connections:
- net 0 V: now also PS3.5 (-VOUT)
- net 12V: now also F12.1, F13.1, F14.1, F4.1, F6.1, F7.1, J7.1, J7.2, J7.3, J7.4; no longer C1.1, C3.2
- net 24 V: now also PS3.3 (+VOUT)
- net GND: now also C5.1, C6.2 (-), J14.3, J14.4, J2.4, J2.5, J2.6, J7.5, J7.6, J7.7, J7.8, PS3.2 (-VIN_(GND)), PS4.2 (ON/OFF_CONTROL), PS4.3 (VIN(-)); no longer J6.1
- net MB: now also F4.2, J2.1, J2.2, J2.3
- net laser: now also F6.2
- net pc: now also F7.2, J14.1, J14.2
- net pol_p: now also F14.2
- net peltier renamed cctrl
- net cctrl: now also C7.2, C8.1, D8.1 (K), F5.1
- new net: C1.1, C3.2, F13.2, PS3.1 (+VIN_(VCC))
- new net GND_cctrl: C7.1, C8.2, D8.2 (A), J6.1, PS4.4 (VOUT(-)), PS4.5 (SENSE(-))
- new net SENS_P: F5.2, PS4.7 (SENSE(+)), PS4.8 (VOUT(+))
- new net vin+_120w: C5.2, C6.1 (+), F12.2, PS4.1 (VIN(+))
- no-connect marks 0 -> 3
Other:
- note added: "LASER: 12V / 1.6A *2"
- note added: "MB: 12V / 2.5A"
- note added: "cool_ctrl: 24V / 3 A"
- note removed: "A voir possible petit"
- note removed: "LASER: 12V / 1.6A"
- note removed: "MB: 12V / 8A"
- note removed: "cool_ctrl: 12V / 10 A"
- moved on the sheet: C1, C18, C19, C2, C20, C21, C22, C23, C24, C25, C26, C3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

Commit message: update computer fuse
Parts:
- removed F7: 8A S.B, 0ABB8000TM, symbol 0ABB-8000-TM:0ABB-8000-TM
- added F7: 10 A S.B, FUSC3216X90N, symbol SF-1206S1000R-2:SF-1206S1000R-2
Connections:
- net 12V: now also F7.1
- net pc: now also F7.2
Other:
- note added: "PC 12 V / 4 A"
- note removed: "PC 12 V / 10 A"
Changed lines of the file:
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@@
+    (stroke (width 0) (type default))
+  )
+  (wire (pts (xy 189.738 115.57) (xy 193.4718 115.57))
     (stroke (width 0) (type default))
   )
@@
     (stroke (width 0) (type default))
   )
-  (wire (pts (xy 189.738 115.57) (xy 193.675 115.57))
-    (stroke (width 0) (type default))
-  )
   (wire (pts (xy 27.686 72.644) (xy 25.146 72.644))
     (stroke (width 0) (type default))
@@
     (stroke (width 0) (type default))
   )
+  (wire (pts (xy 211.2518 115.57) (xy 218.821 115.57))
+    (stroke (width 0) (type default))
+  )
   (wire (pts (xy 31.369 135.255) (xy 34.798 135.255))
     (stroke (width 0) (type default))
@@
     (stroke (width 0) (type default))
   )
-  (wire (pts (xy 211.455 115.57) (xy 218.821 115.57))
-    (stroke (width 0) (type default))
-  )
   (wire (pts (xy 278.257 109.093) (xy 257.937 109.093))
     (stroke (width 0) (type default))
@@
     (stroke (width 0) (type default))
   )
-  (text " PC 12 V / 10 A " (at 252.349 112.268 0)
+  (text " PC 12 V / 4 A " (at 252.349 112.268 0)
     (effects (font (size 1.27 1.27)) (justify right bottom))
   )
@@
     )
   )
+  (symbol (lib_id "SF-1206S1000R-2:SF-1206S1000R-2") (at 193.4718 115.57 0) (unit 1)
+    (in_bom yes) (on_board yes) (dnp no) (fields_autoplaced)
+    (property "Reference" "F7" (at 202.3618 109.22 0)
+      (effects (font (size 1.27 1.27)))
+    )
+    (property "Value" "10 A S.B" (at 202.3618 111.76 0)
+      (effects (font (size 1.27 1.27)))
+    )
+    (property "Footprint" "FUSC3216X90N" (at 207.4418 211.76 0)
+      (effects (font (size 1.27 1.27)) (justify left top) hide)
+    )
+    (property "Datasheet" "https://www.bourns.com/docs/Product-Datasheets/SF-1206S-R.pdf" (at 207.4418 311.76 0)
+      (effects (font (size 1.27 1.27)) (justify left top) hide)
+    )
+    (property "Height" "0.9" (at 207.4418 511.76 0)
+      (effects (font (size 1.27 1.27)) (justify left top) hide)
+    )
+    (property "Mouser Part Number" "652-SF-1206S1000R-2" (at 207.4418 611.76 0)
+      (effects (font (size 1.27 1.27)) (justify left top) hide)
+    )
+    (property "Mouser Price/Stock" "https://www.mouser.co.uk/ProductDetail/Bourns/SF-1206S1000R-2?qs=QpmGXVUTftGXxpZRDDQNPQ%3D%3D" (at 207.4418 711.76 0)
+      (effects (font (size 1.27 1.27)) (justify left top) hide)
+    )
+    (property "Manufacturer_Name" "Bourns" (at 207.4418 811.76 0)
+      (effects (font (size 1.27 1.27)) (justify left top) hide)
+    )
+    (property "Manufacturer_Part_Number" "SF-1206S1000R-2" (at 207.4418 911.76 0)
+      (effects (font (size 1.27 1.27)) (justify left top) hide)
+    )
+    (pin "1")
+    (pin "2")
+    (instances
+      (project "supply_interface"
+        (path "/12450609-d3de-4dca-9e67-f62c6ea94dc7"
+          (reference "F7") (unit 1)
+        )
+      )
+    )
+  )
   (symbol (lib_id "CL21A226MAYNNNE:CL21A226MAYNNNE") (at 238.506 160.655 90) (unit 1)
     (in_bom yes) (on_board yes) (dnp no)
@@
         )
       )
-    )
-  )
-  (symbol (lib_id "0ABB-8000-TM:0ABB-8000-TM") (at 193.675 115.57 0) (unit 1)
-    (in_bom yes) (on_board yes) (dnp no) (fields_autoplaced)
-    (property "Reference" "F7" (at 202.565 109.22 0)
-      (effects (font (size 1.27 1.27)))
-    )
-    (property "Value" "8A S.B" (at 202.565 111.76 0)
-      (effects (font (size 1.27 1.27)))
-    )
-    (property "Footprint" "0ABB8000TM" (at 207.645 211.76 0)
-      (effects (font (size 1.27 1.27)) (justify left top) hide)
-    )
-    (property "Datasheet" "https://www.belfuse.com/resources/datasheets/circuitprotection/ds-CP-0ABB-series.pdf" (at 207.645 311.76 0)
-      (effects (font (size 1.27 1.27)) (justify left top) hide)
-    )
-    (property "Height" "0.56" (at 207.645 511.76 0)
-      (effects (font (size 1.27 1.27)) (justify left top) hide)
-    )
-    (property "Mouser Part Number" "530-0ABB-8000-TM" (at 207.645 611.76 0)
-      (effects (font (size 1.27 1.27)) (justify left top) hide)
-    )
-    (property "Mouser Price/Stock" "https://www.mouser.co.uk/ProductDetail/Bel-Fuse/0ABB-8000-TM?qs=Wj%2FVkw3K%252BMB%2Fdij68u0w3Q%3D%3D" (at 207.645 711.76 0)
-      (effects (font (size 1.27 1.27)) (justify left top) hide)
-    )
-    (property "Manufacturer_Name" "BelFuse" (at 207.645 811.76 0)
-      (effects (font (size 1.27 1.27)) (justify left top) hide)
-    )
-    (property "Manufacturer_Part_Number" "0ABB-8000-TM" (at 207.645 911.76 0)
-      (effects (font (size 1.27 1.27)) (justify left top) hide)
-    )
-    (pin "1")
-    (pin "2")
-    (instances
-      (project "supply_interface"
-        (path "/12450609-d3de-4dca-9e67-f62c6ea94dc7"
-          (reference "F7") (unit 1)
-        )
-      )

Commit message: Update J14
Parts:
- removed J14: 39-28-1043, 39-28-1043, symbol 39-28-1043:39-28-1043
- added J14: 39-30-1041, 39-30-104Y, symbol 39-30-1041:39-30-1041
Connections:
- net GND: now also J14.1, J14.2
- net pc: now also J14.3, J14.4
Changed lines of the file:
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@@
   (junction (at 124.46 109.093) (diameter 0) (color 0 0 0 0)
   )
-  (junction (at 257.937 120.015) (diameter 0) (color 0 0 0 0)
-  )
   (junction (at 53.086 82.804) (diameter 0) (color 0 0 0 0)
   )
@@
   (junction (at 24.511 85.344) (diameter 0) (color 0 0 0 0)
   )
+  (junction (at 257.937 120.015) (diameter 0) (color 0 0 0 0)
+  )
   (junction (at 78.486 162.941) (diameter 0) (color 0 0 0 0)
   )
@@
     (stroke (width 0) (type default))
   )
+  (wire (pts (xy 257.937 120.015) (xy 257.937 124.333))
+    (stroke (width 0) (type default))
+  )
   (wire (pts (xy 238.506 164.719) (xy 238.506 160.655))
     (stroke (width 0) (type default))
@@
     (stroke (width 0) (type default))
   )
-  (wire (pts (xy 257.937 120.015) (xy 257.937 124.333))
+  (wire (pts (xy 257.937 118.11) (xy 257.937 120.015))
     (stroke (width 0) (type default))
   )
@@
     (stroke (width 0) (type default))
   )
-  (wire (pts (xy 257.937 118.11) (xy 257.937 120.015))
-    (stroke (width 0) (type default))
-  )
   (wire (pts (xy 111.379 69.215) (xy 111.379 101.6))
     (stroke (width 0) (type default))
@@
     )
   )
-  (symbol (lib_id "39-28-1043:39-28-1043") (at 257.937 117.475 0) (unit 1)
-    (in_bom yes) (on_board yes) (dnp no) (fields_autoplaced)
-    (property "Reference" "J14" (at 268.097 110.49 0)
-      (effects (font (size 1.27 1.27)))
-    )
-    (property "Value" "39-28-1043" (at 268.097 113.03 0)
-      (effects (font (size 1.27 1.27)))
-    )
-    (property "Footprint" "39-28-1043" (at 274.447 114.935 0)
-      (effects (font (size 1.27 1.27)) (justify left) hide)
-    )
-    (property "Datasheet" "https://www.molex.com/pdm_docs/sd/039281023_sd.pdf" (at 274.447 117.475 0)
-      (effects (font (size 1.27 1.27)) (justify left) hide)
-    )
-    (property "Description" "Mini-Fit Jr. Vertical Header, 4.20mm Pitch, Dual Row, 4 Circuits, without Snap-in Plastic Peg PCB Lock, Tin, Natural" (at 274.447 120.015 0)
-      (effects (font (size 1.27 1.27)) (justify left) hide)
-    )
-    (property "Height" "12.8" (at 274.447 122.555 0)
-      (effects (font (size 1.27 1.27)) (justify left) hide)
-    )
-    (property "Mouser Part Number" "538-39-28-1043" (at 274.447 125.095 0)
-      (effects (font (size 1.27 1.27)) (justify left) hide)
-    )
-    (property "Mouser Price/Stock" "https://www.mouser.co.uk/ProductDetail/Molex/39-28-1043?qs=LQQHZ4xw2XCMHoV0KRLGhg%3D%3D" (at 274.447 127.635 0)
-      (effects (font (size 1.27 1.27)) (justify left) hide)
-    )
-    (property "Manufacturer_Name" "Molex" (at 274.447 130.175 0)
-      (effects (font (size 1.27 1.27)) (justify left) hide)
-    )
-    (property "Manufacturer_Part_Number" "39-28-1043" (at 274.447 132.715 0)
-      (effects (font (size 1.27 1.27)) (justify left) hide)
-    )
-    (pin "1")
-    (pin "2")
-    (pin "3")
-    (pin "4")
-    (instances
-      (project "supply_interface"
-        (path "/12450609-d3de-4dca-9e67-f62c6ea94dc7"
-          (reference "J14") (unit 1)
-        )
-      )
-    )
-  )
   (symbol (lib_id "ATV02W150-HF:ATV02W150-HF") (at 215.646 85.725 270) (unit 1)
     (in_bom yes) (on_board yes) (dnp no)
@@
         )
       )
+    )
+  )
+  (symbol (lib_id "39-30-1041:39-30-1041") (at 257.937 117.475 0) (unit 1)
+    (in_bom yes) (on_board yes) (dnp no) (fields_autoplaced)
+    (property "Reference" "J14" (at 268.097 110.49 0)
+      (effects (font (size 1.27 1.27)))
+    )
+    (property "Value" "39-30-1041" (at 268.097 113.03 0)
+      (effects (font (size 1.27 1.27)))
+    )
+    (property "Footprint" "39-30-104Y" (at 274.447 212.395 0)
+      (effects (font (size 1.27 1.27)) (justify left top) hide)
+    )
+    (property "Datasheet" "https://www.molex.com/pdm_docs/sd/039300020_sd.pdf" (at 274.447 312.395 0)
+      (effects (font (size 1.27 1.27)) (justify left top) hide)
+    )
+    (property "Height" "10" (at 274.447 512.395 0)
+      (effects (font (size 1.27 1.27)) (justify left top) hide)
+    )
+    (property "Mouser Part Number" "538-39-30-1041" (at 274.447 612.395 0)
+      (effects (font (size 1.27 1.27)) (justify left top) hide)
+    )
+    (property "Mouser Price/Stock" "https://www.mouser.co.uk/ProductDetail/Molex/39-30-1041?qs=tRPrwvvr%2FujuCDagC9gKwg%3D%3D" (at 274.447 712.395 0)
+      (effects (font (size 1.27 1.27)) (justify left top) hide)
+    )
+    (property "Manufacturer_Name" "Molex" (at 274.447 812.395 0)
+      (effects (font (size 1.27 1.27)) (justify left top) hide)
+    )
+    (property "Manufacturer_Part_Number" "39-30-1041" (at 274.447 912.395 0)
+      (effects (font (size 1.27 1.27)) (justify left top) hide)
+    )
+    (pin "4")
+    (pin "2")
+    (pin "1")
+    (pin "3")
+    (instances
+      (project "supply_interface"
+        (path "/12450609-d3de-4dca-9e67-f62c6ea94dc7"
+          (reference "J14") (unit 1)
+        )
+      )

Commit message: Update board_shape
Parts:
- removed F5: 4A S.B, FUSC1005X61N, symbol SF-0402S400M-2:SF-0402S400M-2
- removed J14: 39-30-1041, 39-30-104Y, symbol 39-30-1041:39-30-1041
- removed J4: MBES-152, CONN_MBES-152_ALT, symbol MBES-152:MBES-152
- added F5: 4A S.B, FUSC1608X55N, symbol SF-0603S400-2:SF-0603S400-2
- added J14, J3: 39-28-1043, 39-28-1043, symbol 39-28-1043:39-28-1043
Connections:
- net 12V: now also J7.5, J7.6, J7.7, J7.8; no longer J7.1, J7.2, J7.3, J7.4
- net GND: now also J2.1, J2.2, J2.3, J7.1, J7.2, J7.3, J7.4, J14.1, J14.2, J3.1, J3.2; no longer J2.4, J2.5, J2.6, J7.5, J7.6, J7.7, J7.8
- net MB: now also J2.4, J2.5, J2.6; no longer J2.1, J2.2, J2.3
- net SENS_P: now also F5.2
- net cctrl: now also F5.1
- net laser: now also J3.3, J3.4
- net pc: now also J14.3, J14.4
